File: Kicad/PE-Keyboard/KeyboardMatrix.kicad_sch (KiCad schematic)
At the start: 0 parts

Commit message: Started Sch and PCB
Laid out the buttons/Encoder. Chose a nice crystal, realized a connector in board gives challenges with routing.
Parts:
- added D1, D2, D3, D4, D5, D6, D7, D8, D9: 1N4148, Diode_SMD:D_SOD-123, symbol Diode:1N4148
- added SW1, SW2, SW3, SW4, SW6, SW7, SW8, SW9: SW_Push, Button_Switch_Keyboard:SW_Cherry_MX_1.00u_PCB, symbol Switch:SW_Push
- added SW5: RotaryEncoder_Switch, Rotary_Encoder:RotaryEncoder_Alps_EC11E-Switch_Vertical_H20mm, symbol Device:RotaryEncoder_Switch
Connections:
- new net: D1.2 (A), SW1.1
- new net: D3.2 (A), SW3.1
- new net: D9.2 (A), SW9.1
- new net: D6.2 (A), SW6.1
- new net: D4.2 (A), SW4.1
- new net: D8.2 (A), SW8.1
- new net: D5.2 (A), SW5.S2
- new net: D2.2 (A), SW2.1
- new net: D7.2 (A), SW7.1
- new net Col0: D1.1 (K), D6.1 (K)
- new net Col1: D2.1 (K), D7.1 (K)
- new net Col2: D3.1 (K), D8.1 (K)
- new net Col3: D4.1 (K), D9.1 (K)
- new net Col4: D5.1 (K)
- new net Enc0_A: SW5.A
- new net Enc0_B: SW5.B
- new net GND: SW5.C
- new net Row0: SW1.2, SW2.2, SW3.2, SW4.2, SW5.S1
- new net Row1: SW6.2, SW7.2, SW8.2, SW9.2
